File: schematics/desk.kicad_sch (KiCad schematic)
At the start: 42 parts, among them J1 in motor housing, mates with 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, J2 to motor housing, mates with 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, J3 to handset, mates with J4, J4 in handset, mates with J3, K1 energized = UP (raises desk), K2 energized = DOWN (lowers desk), M1 2R5 winding, Q1 IRLB8721, Q2 2N7002, Q3 2N7002, Q4 BC337, Q5 BC327, SW1 DOWN rocker, SW2 UP rocker, SW3 top limit, SW4 bottom limit, U1 LM2596HV 29V-5V, U2 ESP32, U3 74HC123 250ms, U5 ACS724xLCTR-05AB, U6 74HC08

Commit message: Fix Q1 to IRLZ44N (30V IRLB8721 didn't clear the 29-30V rail)
Caught by cross-checking HANDOFF.md item 7 against the actual repo:
Q1 was still IRLB8721 despite being flagged for this exact fix (30V
VDSS, flyback clamping puts it at/over absolute max every cycle on a
29V nominal / 30V unloaded rail). The other half of item 7 - symbols.py
existing with no exec() - did hold.

Also recorded item 6 as resolved rather than open: the current sensor
choice HANDOFF called "not yet decided" was already committed in the
schematic (ACS724xLCTR-05AB, bidirectional 5A - exactly its own stated
requirements) and assumed by README §4.4. Updated README §6 BOM/§6.2 to
match current reality (IRLZ44N, discrete BC337/BC327 driver instead of
the stale TC4427 IC reference) and added a §5 correction entry.
Parts:
- Q1: value IRLB8721 -> IRLZ44N
Changed lines of the file:
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@@
     (in_bom yes) (on_board yes) (dnp no)
     (property "Reference" "Q1" (at 397.51 328.93 0) (effects (font (size 1.27 1.27)) (justify left)))
-    (property "Value" "IRLB8721" (at 397.51 331.47 0) (effects (font (size 1.0 1.0)) (justify left)))
+    (property "Value" "IRLZ44N" (at 397.51 331.47 0) (effects (font (size 1.0 1.0)) (justify left)))
     (property "Footprint" "" (at 392.43 330.20 0) (effects (font (size 1.27 1.27)) hide))
     (property "Datasheet" "" (at 392.43 330.20 0) (effects (font (size 1.27 1.27)) hide))

Commit message: Add board-side screw terminals, resolve remaining HANDOFF.md items
Screw terminal redesign: J2/J3 (board-side Mini-Fit connectors) are
dropped from the schematic entirely, replaced by four 2-position screw
terminals (TB1-TB4) - the board now only ever solders to a screw
terminal, no crimp tool needed for board assembly; a short pigtail
carries each pair on to the actual Mini-Fit (J1/J4, unchanged). TB2/TB4
mirrored so their pins face where their wires actually go, and moved
clear of TB1/TB3 now that they're not physically one connector anymore.
J1/J4 labels split across two lines (esc() extended to support literal
newlines in Kicad property text - a small general capability, not
J1/J4-specific).

HANDOFF.md items 1 and 2 resolved: Q2/Q3 2N7002 -> 2N7000 (BOM row
added), and the 74HC122-vs-74HC123 investigation recorded in APPENDIX
§5.7 as a negative result so it isn't re-researched later.

NETLIST.md brought back in sync with the actual schematic: TB1-4,
corrected Q1/Q2/Q3 values, corrected K1/K2 A1/A2 coil-pin assignment
(stale since the earlier relay rotation, not something today's changes
caused), ESP32 display correction. README §6 gained BOM rows for the
screw terminals and flyback diodes and a §6.4 note on the pigtail
arrangement.

Verified: 0 candidate shorts, 0 diagonal segments, same 15
crossings/6 body-crossings baseline as before (all previously triaged
as benign), ERC steady at 129 violations (net +2 from the expected
lib_symbol_issues warning on each new TB, minus 2 removed with J2/J3).
Parts:
- removed J2: to motor housing, mates with J1, symbol L:Conn_02x02_Top_Bottom
- added TB1: motor pair, symbol L:Screw_Terminal_01x02
- added TB2: supply pair, symbol L:Screw_Terminal_01x02
- added TB4: power pair, symbol L:Screw_Terminal_01x02
- J1: value in motor housing, mates with J2 -> in motor housing mates with board pigtail (TB1/TB2)
- J4: value in handset, mates with J3 -> in handset mates with board pigtail (TB3/TB4)
- Q2, Q3: value 2N7002 -> 2N7000
- TB3: renamed from J3; value to handset, mates with J4 -> signal pair; symbol L:Conn_02x02_Top_Bottom -> L:Screw_Terminal_01x02
Connections:
- net +3V3: now also TB4.1 (Pin_1); no longer TB3.3 (Pin_3)
- net GND: now also TB2.2 (Pin_2), TB4.2 (Pin_2); no longer TB3.4 (Pin_4)
- net at K2.11: now also TB1.1 (Pin_1)
- net at U5.1 (IP+), U5.2 (IP+): now also TB1.2 (Pin_2)
- net at C1.1, D1.1, U1.1 (VIN): now also TB2.1 (Pin_1)

Commit message: Assign PCB footprints to every on-board part
schlib.py: place() gains footprint= (override) and on_board= params;
Sym now carries a per-symbol-type default footprint, set once in
symbols.py rather than repeated at every call site (same pattern as
ref_dy/val_dy). Per-instance overrides used where package size differs
within one symbol type (C1/C2 electrolytic vs C3 ceramic, D5 Schottky
vs D2/D3/D4/D6 signal diodes, Q1 TO-220 vs Q2/Q3 TO-92).

The 10 parts that live in the motor housing/handset/wall supply - not
on this board - are marked on_board=False (M1, J1, J4, PSU1, SW1-4,
D3/D4) so "Update PCB from Schematic" won't try to place them.

Two footprints are placeholders pending the physical part: the ESP32
devkit (generic 2x22 pin socket - real DevKitC row spacing varies by
board width) and the ACS724 carrier (generic 1x8 pin socket). The
relay footprint (SANYOU SRD-series) is the closest available match to
the Songle part named in the BOM - verify against its datasheet before
fabrication.

Fixed a design/doc inconsistency found while assigning these: README
§6.3 and the BOM assumed a driver-included relay module (checking
active-high/low, JD-VCC jumper), but the schematic drives the bare
relay coil directly with its own Q2/Q3/D2/D6 circuit - a module would
make that circuit redundant. Rewrote §6.3 and the BOM row accordingly,
and retired the now-moot "relay polarity unverified" item from
CLAUDE.md/TODO.md/README §9 - boot-safety is by construction (R1/R2/R6
hold Q2/Q3 off at boot, same as the existing brake-state invariant).
Also corrected §6.5's package table: LM2596HV and the relay are bare
through-hole parts, not modules: only the ESP32 devkit and ACS724
carrier genuinely are.
Parts:
- C1: footprint (none) -> Capacitor_THT:CP_Radial_D10.0mm_P5.00mm
- C2: footprint (none) -> Capacitor_THT:CP_Radial_D8.0mm_P3.50mm
- C3: footprint (none) -> Capacitor_THT:C_Disc_D5.0mm_W2.5mm_P5.00mm
- D1: footprint (none) -> Diode_THT:D_DO-15_P10.16mm_Horizontal
- D2, D3, D4, D6: footprint (none) -> Diode_THT:D_DO-35_SOD27_P7.62mm_Horizontal
- D5: footprint (none) -> Diode_THT:D_DO-201AD_P12.70mm_Horizontal
- K1, K2: footprint (none) -> Relay_THT:Relay_SPDT_SANYOU_SRD_Series_Form_C
- Q1: footprint (none) -> Package_TO_SOT_THT:TO-220-3_Vertical
- Q2, Q3, Q4, Q5: footprint (none) -> Package_TO_SOT_THT:TO-92_Inline
- R1, R11, R13, R14, R15, R2, R3, R4, R5, R6, R7: footprint (none) -> Resistor_THT:R_Axial_DIN0207_L6.3mm_D2.5mm_P10.16mm_Horizontal
- TB1, TB2, TB3, TB4: footprint (none) -> TerminalBlock:TerminalBlock_MaiXu_MX126-5.0-02P_1x02_P5.00mm
- U1: footprint (none) -> Package_TO_SOT_THT:TO-220-5_Vertical
- U2: footprint (none) -> Connector_PinSocket_2.54mm:PinSocket_2x22_P2.54mm_Vertical
- U3: footprint (none) -> Package_DIP:DIP-16_W7.62mm
- U5: footprint (none) -> Connector_PinSocket_2.54mm:PinSocket_1x08_P2.54mm_Vertical
- U6: footprint (none) -> Package_DIP:DIP-14_W7.62mm

Commit message: Reference: single-board schematic before the logic/power PCB split
Snapshot of the design right before splitting into two boards - U2
(ESP32) off-board via JP1/JP2/JP3 pigtails (mated by JP4/JP5/JP6), but
the watchdog-gated drive signals still wire straight from U6 into
Q2/Q3/R7, and ISENSE still rides JP4's own pigtail to the ESP32, both
as plain same-board wires (no JP7-JP12 board-tie connectors).

Kept as a fallback in case the board-split-plus-jumpers experiment
(continuing on main) doesn't pan out. NETLIST.md/README.md are not
refreshed for this snapshot - schematics/gen/sch.py is the source of
truth per its own header.
Parts:
- removed R6: 10k, Resistor_THT:R_Axial_DIN0207_L6.3mm_D2.5mm_P10.16mm_Horizontal, symbol L:R
- added JP1, JP5: drive pigtail, Connector_JST:JST_XH_B4B-XH-A_1x04_P2.50mm_Vertical, symbol L:Conn_01x04
- added JP2, JP4: sense pigtail, Connector_JST:JST_XH_B3B-XH-A_1x03_P2.50mm_Vertical, symbol L:Conn_01x03
- added JP3, JP6: power pigtail, Connector_JST:JST_XH_B3B-XH-A_1x03_P2.50mm_Vertical, symbol L:Conn_01x03
- added Q3: 2N7000, Package_TO_SOT_THT:TO-92_Wide, symbol L:Q_NMOS_GDS
- K1, K2: footprint Relay_THT:Relay_SPDT_SANYOU_SRD_Series_Form_C -> Relay_THT:Relay_SPDT_Hongfa_JQC-3FF_0XX-1Z
- Q2, Q4, Q5: footprint Package_TO_SOT_THT:TO-92_Inline -> Package_TO_SOT_THT:TO-92_Wide
- R6: renamed from Q3; value 2N7000 -> 10k; footprint Package_TO_SOT_THT:TO-92_Inline -> Resistor_THT:R_Axial_DIN0207_L6.3mm_D2.5mm_P10.16mm_Horizontal; symbol L:Q_NMOS_GDS -> L:R
Connections:
- net +3V3: now also JP3.2 (Pin_2), JP6.2 (Pin_2)
- net +5V: now also JP3.1 (Pin_1), JP6.1 (Pin_1)
- net GND: now also R6.2, JP3.3 (Pin_3), JP6.3 (Pin_3), Q3.3 (S); no longer R6.3 (S)
- net ISENSE: now also JP2.3 (Pin_3), JP4.3 (Pin_3)
- net SW_UP: now reaches R11.1, R13.2, U2.15 (GPIO9/ADC1_CH8)
- net SW_UP: now also JP2.1 (Pin_1), JP4.1 (Pin_1)
- net DIR_B: now reaches R2.1, U6.5
- net DIR_B: now also U2.37 (GPIO40/MTDO), JP1.3 (Pin_3), JP5.3 (Pin_3); no longer U2.11 (GPIO18/ADC2_CH7)
- net DIR_A: now reaches R1.1, U6.2
- net DIR_A: now also U2.36 (GPIO39/MTCK), JP1.2 (Pin_2), JP5.2 (Pin_2); no longer U2.10 (GPIO17/ADC2_CH6)
- net SW_DN: now reaches R14.1, R15.2, U2.16 (GPIO10/ADC1_CH9)
- net SW_DN: now also JP2.2 (Pin_2), JP4.2 (Pin_2)
- net at U2.27 (GPIO21): no longer U6.10
- net PWM: now reaches U2.39 (GPIO42/MTMS)
- net PWM: now also R6.1, U6.10, JP1.4 (Pin_4), JP5.4 (Pin_4)
- net KICK: now reaches U2.4 (GPIO4/ADC1_CH3)
- net KICK: now also U3.1 (A), JP1.1 (Pin_1), JP5.1 (Pin_1)
- net at U2.41 (GPIO1/ADC1_CH0): no longer U3.1 (A)
- net at U6.6: now also Q3.1 (G); no longer R6.1 (G)
- net at D6.2 (A), K2.A1: now also Q3.2 (D); no longer R6.2 (D)
Other:
- note added: "HANDSET INTERFACE"
- note added: "U2 PIGTAILS"

Commit message: Long shot: bring U2 back on-board - works, once its footprint is fixed
Removed the off-board ESP32 pigtail arrangement (JP1/JP2/JP3, and the
JP4/JP5/JP6 on-board mates - kept in the schematic as on_board=False
since their own wiring still anchors TB3/TB4/R11/R13/R14/R15's layout)
and placed U2 directly on the board instead, wired straight to U3/U6/
the rocker dividers/R4-R5 by matching label, the same mechanism WDOG
already uses. Board expanded to 194x150mm to fit U2's real footprint.

First attempt used the existing MCU.footprint - a generic 2x22 header
with both rows only 2.54mm apart - and Freerouting got stuck at 9/68
nets unrouted after 10 passes and 100+GB allocated, a real regression
from the off-board board's clean 1-via result. Turned out to be the
footprint, not U2's presence: that symbol's own comment already flagged
it as "a generic dual-row placeholder" needing the real DevKitC's row
spacing - which is 1 inch (25.4mm), not 2.54mm (confirmed against a
real board's dimension drawing). A 2.54mm-spaced 44-pin footprint is a
solid wall to a router; a real connector has a channel down the middle.

Built the correct footprint (two PinSocket_1x22_P2.54mm's, 25.4mm
apart - local.pretty/, wired up via fp-lib-table) and re-routed: 9
seconds, 0/68 unrouted, 3 vias, DRC clean except one pre-existing-style
GND-to-pour-zone gap on D1 (same minor category seen on other branches,
not a routing failure). Comparable to the off-board result (1 via) and
nothing like the stuck 9-unrouted state the wrong footprint produced.

Conclusion: U2 CAN come back on-board without real cost, given a
correctly-dimensioned footprint - the earlier "doesn't work" finding
was an artifact of bad footprint data, not board density. Pin-to-side
numbering (1-22/23-44) is still a placeholder pending the real board's
own silkscreen/datasheet.
Parts:
- removed C1: 220u 50V, Capacitor_THT:CP_Radial_D10.0mm_P5.00mm, symbol L:C
- removed JP1, JP5: drive pigtail, Connector_JST:JST_XH_B4B-XH-A_1x04_P2.50mm_Vertical, symbol L:Conn_01x04
- removed JP2: sense pigtail, Connector_JST:JST_XH_B3B-XH-A_1x03_P2.50mm_Vertical, symbol L:Conn_01x03
- removed JP3, JP6: power pigtail, Connector_JST:JST_XH_B3B-XH-A_1x03_P2.50mm_Vertical, symbol L:Conn_01x03
- removed SW2: UP rocker, symbol L:SW_Push_SPDT
- removed SW3: top limit, symbol L:SW_Push_Open
- removed unit 1 of U3
- removed unit 5 of U6
- added C2: 220u 10V, Capacitor_THT:CP_Radial_D8.0mm_P3.50mm, symbol L:C
- added D3: allows down, Diode_THT:D_DO-35_SOD27_P7.62mm_Horizontal, symbol L:D
- added D6: flyback, Diode_THT:D_DO-35_SOD27_P7.62mm_Horizontal, symbol L:D
- added R1: 10k, Resistor_THT:R_Axial_DIN0207_L6.3mm_D2.5mm_P10.16mm_Horizontal, symbol L:R
- added TB4: power pair, TerminalBlock:TerminalBlock_MaiXu_MX126-5.0-02P_1x02_P5.00mm, symbol L:Screw_Terminal_01x02
- added U5: ACS724xLCTR-05AB, Connector_PinSocket_2.54mm:PinSocket_1x08_P2.54mm_Vertical, symbol L:ACS712xLCTR-05B
- C1: renamed from U5; value ACS724xLCTR-05AB -> 220u 50V; footprint Connector_PinSocket_2.54mm:PinSocket_1x08_P2.54mm_Vertical -> Capacitor_THT:CP_Radial_D10.0mm_P5.00mm; symbol L:ACS712xLCTR-05B -> L:C
- JP6: renamed from D6; value flyback -> power pigtail; footprint Diode_THT:D_DO-35_SOD27_P7.62mm_Horizontal -> Connector_JST:JST_XH_B3B-XH-A_1x03_P2.50mm_Vertical; symbol L:D -> L:Conn_01x03
- SW2: renamed from D3; value allows down -> UP rocker; footprint Diode_THT:D_DO-35_SOD27_P7.62mm_Horizontal -> (none); symbol L:D -> L:SW_Push_SPDT
- SW3: renamed from C2; value 220u 10V -> top limit; footprint Capacitor_THT:CP_Radial_D8.0mm_P3.50mm -> (none); symbol L:C -> L:SW_Push_Open
- U2: footprint Connector_PinSocket_2.54mm:PinSocket_2x22_P2.54mm_Vertical -> local:DevKitC_2x22_P2.54mm_1in_row
- U3: renamed from TB4; value power pair -> 74HC123 250ms; footprint TerminalBlock:TerminalBlock_MaiXu_MX126-5.0-02P_1x02_P5.00mm -> Package_DIP:DIP-16_W7.62mm; symbol L:Screw_Terminal_01x02 -> L:74LS123
- U6: renamed from R1; value 10k -> 74HC08; footprint Resistor_THT:R_Axial_DIN0207_L6.3mm_D2.5mm_P10.16mm_Horizontal -> Package_DIP:DIP-14_W7.62mm; symbol L:R -> L:74LS08
Connections:
- net +3V3: now also JP6.2 (Pin_2), TB4.1 (Pin_1); no longer U3.1 (Pin_1)
- net +5V: now also U3.2 (B), U3.3 (Clr), U6.14 (VCC), C2.1, D6.1 (K), U5.8 (VCC); no longer C1.8 (VCC), SW3.1
- net DIR_A: now also R1.1; no longer U6.1
- net DRV_UP: now also U5.3 (IP-), U5.4 (IP-); no longer C1.3 (IP-), C1.4 (IP-)
- net GND: now also C1.2, JP6.3 (Pin_3), U6.7 (GND), C2.2, R1.2, TB4.2 (Pin_2), U5.5 (GND); no longer C1.5 (GND), SW3.2, U3.2 (Pin_2), U6.2
- net KICK: now also U3.1 (A)
- net WDOG: now also U3.13 (Q)
- net at D1.1, TB2.1 (Pin_1), U1.1 (VIN): now also C1.1
- net at C3.2, R3.2: now also U3.14 (Cext), U3.15 (RCext)
- net at J1.1 (Pin_1): now also SW3.2 (B), D3.1 (K); no longer SW2.1 (K)
- net at J4.1 (Pin_1): now also SW2.2 (B)
- net at J4.3 (Pin_3), SW1.1 (A): now also SW2.1 (A)
- net at J4.4 (Pin_4), SW1.3 (C): now also SW2.3 (C)
- net at R4.1: now also U5.7 (VIOUT); no longer C1.7 (VIOUT)
- net at K2.A1, Q3.2 (D): now also D6.2 (A); no longer JP6.2 (A)
- net at M1.1 (+): now also SW3.1 (A), D3.2 (A); no longer SW2.2 (A)
- new net: TB1.2 (Pin_2), U5.1 (IP+), U5.2 (IP+)
Other:
- note removed: "U2 PIGTAILS"

Commit message: Drop the ACS724 Pololu carrier for a bare chip, draw the pigtail plugs, and clear the drawing-sheet border
ACS724 moves from the Pololu carrier to a bare SOIC-8 chip on a generic
SOIC-8-to-DIP-8 adapter. That drops two caps the carrier used to provide
for free - a 0.1uF VCC bypass and a 1nF FILTER-to-GND cap, both confirmed
against Allegro's own ACS712/ACS724 application circuit - so they're now
discrete parts on the main board (C4, C5), placed and routed. README,
SHOPPING_LIST.md and NETLIST.md are reconciled with the swap.

D1 goes back to a horizontal/laid-flat DO-15 mount now that the board has
room again, instead of the standing 2.54mm-pitch mount from the earlier
space crunch - easier to mount, and it drops D1's height off the board.

J2/J3 are now drawn as real parts: the pigtail's own Mini-Fit Jr plugs,
crimped onto the cable, distinct from J1/J4's fixed receptacles in the
motor housing/handset. Previously only J1/J4 were drawn, with TB1-4
connected to them purely by matching net-name labels and no literal
component in between - electrically fine, but understated what's
actually a real, separate, buy-and-crimp part. Both are on_board=False,
same as J1/J4/M1/PSU1.

The PCB board outline sat flush with the coordinate origin, which put it
running straight through the drawing sheet's default border margin in
any print/screenshot. Moved the whole board (outline, footprints,
tracks, zones, aux/grid origin) by a uniform +15/+15mm via pcbnew's own
board Move() - a rigid translation, no relative geometry changed - and
updated the handful of literal absolute-coordinate references in
enclosure/shell.scad (the two pigtail wall-hole centers, the USB slot)
to match. The mounting-hole positions are parametric and needed no
change. STL regenerated and re-rendered against the shifted board.

Also moved the aux/grid origin to H1's corner (was an arbitrary point
off the board entirely, left over from before the board was resized).
Parts:
- removed D1: 33V bidir, Diode_THT:D_DO-15_P10.16mm_Horizontal, symbol L:TVS
- removed J1: in motor housing mates with board pigtail (TB1/TB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, symbol L:Conn_02x02_Top_Bottom
- removed JP6: power pigtail, Connector_JST:JST_XH_B3B-XH-A_1x03_P2.50mm_Vertical, symbol L:Conn_01x03
- removed K2: energized = DOWN (lowers desk), Relay_THT:Relay_SPDT_Hongfa_JQC-3FF_0XX-1Z, symbol L:Relay_SPDT
- removed Q4: BC337, Package_TO_SOT_THT:TO-92_Wide, symbol L:Q_NPN_CBE
- removed R5: 20k, Resistor_THT:R_Axial_DIN0207_L6.3mm_D2.5mm_P10.16mm_Horizontal, symbol L:R
- removed TB3: signal pair, TerminalBlock:TerminalBlock_MaiXu_MX126-5.0-02P_1x02_P5.00mm, symbol L:Screw_Terminal_01x02
- removed U3: 74HC123 250ms, Package_DIP:DIP-16_W7.62mm, symbol L:74LS123
- added C3: 2u2, Capacitor_THT:C_Disc_D5.0mm_W2.5mm_P5.00mm, symbol L:C
- added C4: 100n, Capacitor_THT:C_Disc_D5.0mm_W2.5mm_P5.00mm, symbol L:C
- added C5: 1n, Capacitor_THT:C_Disc_D5.0mm_W2.5mm_P5.00mm, symbol L:C
- added D1: 33V bidir, Diode_THT:D_DO-15_P10.16mm_Horizontal, symbol L:D_TVS
- added J2: on pigtail plug crimped here, mates with J1, symbol L:Conn_02x02_Top_Bottom
- added J3: on pigtail plug crimped here, mates with J4, symbol L:Conn_02x02_Top_Bottom
- added PSU1: 29V 1.8A 52W, symbol L:HLK-30M05
- added Q2: 2N7000, Package_TO_SOT_THT:TO-92_Wide, symbol L:Q_NMOS_GDS
- added R3: 100k, Resistor_THT:R_Axial_DIN0207_L6.3mm_D2.5mm_P10.16mm_Horizontal, symbol L:R
- added TB4: power pair, TerminalBlock:TerminalBlock_MaiXu_MX126-5.0-02P_1x02_P5.00mm, symbol L:Screw_Terminal_01x02
- added U5: ACS724xLCTR-05AB, Package_DIP:DIP-8_W7.62mm_Socket, symbol L:ACS712xLCTR-05B
- J1: renamed from PSU1; value 29V 1.8A 52W -> in motor housing mates with board pigtail (TB1/TB2); symbol L:HLK-30M05 -> L:Conn_02x02_Top_Bottom
- K2: renamed from U5; value ACS724xLCTR-05AB -> energized = DOWN (lowers desk); footprint Connector_PinSocket_2.54mm:PinSocket_1x08_P2.54mm_Vertical -> Relay_THT:Relay_SPDT_Hongfa_JQC-3FF_0XX-1Z; symbol L:ACS712xLCTR-05B -> L:Relay_SPDT
- Q4: renamed from Q2; value 2N7000 -> BC337; symbol L:Q_NMOS_GDS -> L:Q_NPN_CBE
- R4: footprint Resistor_THT:R_Axial_DIN0207_L6.3mm_D2.5mm_P10.16mm_Horizontal -> Resistor_THT:R_Axial_DIN0207_L6.3mm_D2.5mm_P2.54mm_Vertical
- R5: renamed from JP4; value sense pigtail -> 20k; footprint Connector_JST:JST_XH_B3B-XH-A_1x03_P2.50mm_Vertical -> Resistor_THT:R_Axial_DIN0207_L6.3mm_D2.5mm_P2.54mm_Vertical; symbol L:Conn_01x03 -> L:R
- TB3: renamed from TB4; value power pair -> signal pair
- U3: renamed from R3; value 100k -> 74HC123 250ms; footprint Resistor_THT:R_Axial_DIN0207_L6.3mm_D2.5mm_P10.16mm_Horizontal -> Package_DIP:DIP-16_W7.62mm; symbol L:R -> L:74LS123
- U3: renamed from C3; value 2u2 -> 74HC123 250ms; footprint Capacitor_THT:C_Disc_D5.0mm_W2.5mm_P5.00mm -> Package_DIP:DIP-16_W7.62mm; symbol L:C -> L:74LS123
Connections:
- net +3V3: now also J4.3 (Pin_3), SW1.1 (A), SW2.1 (A), J3.3 (Pin_3), TB4.1 (Pin_1); no longer TB3.1 (Pin_1)
- net +5V: now also K2.A2, Q4.1 (C), U3.16 (VCC), U3.2 (B), U3.3 (Clr), C4.1, R3.1, U5.8 (VCC); no longer K2.8 (VCC), U3.1
- net DRV_UP: now also U5.3 (IP-), U5.4 (IP-); no longer K2.3 (IP-), K2.4 (IP-)
- net GND: now also J1.4 (Pin_4), J4.4 (Pin_4), R5.2, SW1.3 (C), SW2.3 (C), U3.8 (GND), C3.1, C4.2, C5.2, D1.2 (A2), J2.4 (Pin_4), J3.4 (Pin_4), PSU1.3 (-Vout), Q2.3 (S), TB4.2 (Pin_2), U5.5 (GND); no longer K2.5 (GND), Q4.3 (S), TB3.2 (Pin_2), U3.1
- net KICK: now also U3.1 (A)
- net L: now also PSU1.1 (AC/L); no longer J1.1 (AC/L)
- net MRET: now also K2.14
- net N: now also PSU1.2 (AC/N); no longer J1.2 (AC/N)
- net SW_DN: no longer R5.2 (Pin_2)
- net SW_UP: no longer R5.1 (Pin_1)
- net VSW: now also K2.12
- net WDOG: now also U3.13 (Q)
- net MOT_A: now reaches D3.1 (K), SW3.2 (B)
- net MOT_A: now also J1.1 (Pin_1), K2.11, TB1.1 (Pin_1), J2.1 (Pin_1)
- net at U6.3: now also Q2.1 (G); no longer Q4.1 (G)
- net at Q5.2 (B), R7.2: now also Q4.2 (B)
- net MOT_B: now reaches D4.1 (K), SW4.2 (B)
- net MOT_B: now also J1.2 (Pin_2), TB1.2 (Pin_2), J2.2 (Pin_2), U5.1 (IP+), U5.2 (IP+)
- net at D6.2 (A), Q3.2 (D): now also K2.A1
- net at D2.2 (A), K1.A1: now also Q2.2 (D); no longer Q4.2 (D)
- net +29V_RAW: now reaches C1.1, TB2.1 (Pin_1), U1.1 (VIN)
- net +29V_RAW: now also J1.3 (Pin_3), D1.1 (A1), J2.3 (Pin_3), PSU1.6 (+Vout)
- net HND_A: now reaches R11.2
- net HND_A: now also J4.1 (Pin_1), SW2.2 (B), TB3.1 (Pin_1), J3.1 (Pin_1)
- net HND_B: now reaches R14.2
- net HND_B: now also J4.2 (Pin_2), SW1.2 (B), TB3.2 (Pin_2), J3.2 (Pin_2)
- net at Q1.1 (G), Q5.3 (E): now also Q4.3 (E)
- net VIOUT: now reaches R4.1
- net VIOUT: now also U5.7 (VIOUT); no longer K2.7 (VIOUT)
- net ISENSE: no longer names the net of R4.2, U2.40 (GPIO2/ADC1_CH1)
- net ISENSE: now also R5.1; no longer R5.3 (Pin_3)
- new net: C3.2, R3.2, U3.14 (Cext), U3.15 (RCext)
- new net: C5.1, U5.6 (FILTER)
Other:
- note added: "W1 (cont'd): from J2, elsewhere on this sheet"
- note added: "W1: pigtail, 4-cond, bare wire into TB1/TB2"
- note added: "W2 (cont'd): from J3, elsewhere on this sheet"
- note added: "W2: pigtail, 4-cond, bare wire into TB3/TB4"
- moved on the sheet: TB3
