File: schematics/desk.kicad_sch (KiCad schematic)
At the start: 48 parts, among them J1 in motor housing mates with b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, J2 on pigtail plug crimped here,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, J3 on pigtail plug crimped here,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, J4 in handset mates with board p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, K1 energized = UP (raises desk), K2 energized = DOWN (lowers desk), M1 2R5 winding, Q1 IRLZ44N, Q2 2N7000, Q3 2N7000, Q4 BC337, Q5 BC327, SW1 DOWN rocker, SW2 UP rocker, SW3 top limit, SW4 bottom limit, U1 LM2596HV 29V-5V, U2 ESP32, U3 74HC123 250ms, U5 ACS724xLCTR-05AB, U6 74HC08

Commit message: Fix TB pitch/ToF routing, renumber references, fix stale docs, implement read_current_()
- Fix TB1-5 footprint pitch to match the actually-ordered 2.54mm Degson
  part (board previously used a 5.00mm-pitch footprint)
- Add TB5 for a future ToF sensor's SDA/SCL, moved to GPIO38/41 after
  GPIO12/13 proved unroutable near U1's own margin; +3V3/GND for it
  shares TB2 instead of a dedicated terminal
- Renumber every reference designator (R/C/D/Q/U/TB/J/SW) to match
  schematic reading order, closing all numbering gaps
- Fix several stale references found along the way: leftover per-gate
  IC labels (U8/U9) in the relay-drive chain description, a fuse (F1)
  no longer fitted by design, "relay module" wording where this design
  drives coils directly, two incorrectly-laid-out ASCII diagrams (one
  showing SPDT switches with only 2 of 3 real terminals), and an ACS712
  sensitivity figure inconsistent with its actual datasheet spec
- Confirm §1.6's connector numbering against Molex's real SD-5557-003
  drawing instead of treating it as unverifiable
- Implement read_current_() for both ESP-IDF 4.x and 5.x; fix
  desk.yaml, which targeted the classic ESP32 instead of the S3 this
  design is built around (every GPIO number was consequently wrong)
- Strip SHOPPING_LIST.md down to a plain checklist
Parts:
- removed D1: 33V bidir, Diode_THT:D_DO-15_P10.16mm_Horizontal, symbol L:D_TVS
- removed D4: allows up, Diode_THT:D_DO-35_SOD27_P7.62mm_Horizontal, symbol L:D
- removed J1: in motor housing mates with board pigtail (TB1/TB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, symbol L:Conn_02x02_Top_Bottom
- removed K1: energized = UP (raises desk), Relay_THT:Relay_SPDT_Hongfa_JQC-3FF_0XX-1Z, symbol L:Relay_SPDT
- removed K2: energized = DOWN (lowers desk), Relay_THT:Relay_SPDT_Hongfa_JQC-3FF_0XX-1Z, symbol L:Relay_SPDT
- removed Q1: IRLZ44N, Package_TO_SOT_THT:TO-220-3_Vertical, symbol L:Q_NMOS_GDS
- removed Q2: 2N7000, Package_TO_SOT_THT:TO-92_Wide, symbol L:Q_NMOS_GDS
- removed Q4: BC337, Package_TO_SOT_THT:TO-92_Wide, symbol L:Q_NPN_CBE
- removed Q5: BC327, Package_TO_SOT_THT:TO-92_Wide, symbol L:Q_PNP_CBE
- removed R1, R2, R6: 10k, Resistor_THT:R_Axial_DIN0207_L6.3mm_D2.5mm_P10.16mm_Horizontal, symbol L:R
- removed R3: 100k, Resistor_THT:R_Axial_DIN0207_L6.3mm_D2.5mm_P10.16mm_Horizontal, symbol L:R
- removed SW1: DOWN rocker, symbol L:SW_Push_SPDT
- removed SW2: UP rocker, symbol L:SW_Push_SPDT
- removed SW3: top limit, symbol L:SW_Push_Open
- removed SW4: bottom limit, symbol L:SW_Push_Open
- removed TB1: motor pair, TerminalBlock:TerminalBlock_MaiXu_MX126-5.0-02P_1x02_P5.00mm, symbol L:Screw_Terminal_01x02
- removed TB2: supply pair, TerminalBlock:TerminalBlock_MaiXu_MX126-5.0-02P_1x02_P5.00mm, symbol L:Screw_Terminal_01x02
- removed U3: 74HC123 250ms, Package_DIP:DIP-16_W7.62mm, symbol L:74LS123
- removed U5: ACS724xLCTR-05AB, Package_DIP:DIP-8_W7.62mm_Socket, symbol L:ACS712xLCTR-05B
- removed U6: 74HC08, Package_DIP:DIP-14_W7.62mm, symbol L:74LS08
- added D1: SB560, Diode_THT:D_DO-201AD_P12.70mm_Horizontal, symbol L:D
- added D2: flyback, Diode_THT:D_DO-35_SOD27_P7.62mm_Horizontal, symbol L:D
- added D6: allows up, Diode_THT:D_DO-35_SOD27_P7.62mm_Horizontal, symbol L:D
- added J3: in motor housing mates with board pigtail (TB1/TB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, symbol L:Conn_02x02_Top_Bottom
- added Q1: BC337, Package_TO_SOT_THT:TO-92_Wide, symbol L:Q_NPN_CBE
- added Q2: BC327, Package_TO_SOT_THT:TO-92_Wide, symbol L:Q_PNP_CBE
- added Q4: 2N7000, Package_TO_SOT_THT:TO-92_Wide, symbol L:Q_NMOS_GDS
- added Q5: IRLZ44N, Package_TO_SOT_THT:TO-220-3_Vertical, symbol L:Q_NMOS_GDS
- added R10, R8, R9: 10k, Resistor_THT:R_Axial_DIN0207_L6.3mm_D2.5mm_P10.16mm_Horizontal, symbol L:R
- added R11: 1k, Resistor_THT:R_Axial_DIN0207_L6.3mm_D2.5mm_P10.16mm_Horizontal, symbol L:R
- added SW1: top limit, symbol L:SW_Push_Open
- added SW2: bottom limit, symbol L:SW_Push_Open
- added SW3: DOWN rocker, symbol L:SW_Push_SPDT
- added SW4: UP rocker, symbol L:SW_Push_SPDT
- added TB3: ToF signal pair, TerminalBlock:TerminalBlock_Xinya_XY308-2.54-2P_1x02_P2.54mm_Horizontal, symbol L:Screw_Terminal_01x02
- added TB4: motor pair, TerminalBlock:TerminalBlock_Xinya_XY308-2.54-2P_1x02_P2.54mm_Horizontal, symbol L:Screw_Terminal_01x02
- added TB5: supply pair, TerminalBlock:TerminalBlock_Xinya_XY308-2.54-2P_1x02_P2.54mm_Horizontal, symbol L:Screw_Terminal_01x02
- added U2: 74HC123 250ms, Package_DIP:DIP-16_W7.62mm, symbol L:74LS123
- added U3: 74HC08, Package_DIP:DIP-14_W7.62mm, symbol L:74LS08
- added U4: ACS712ELCTR-05B, Package_DIP:DIP-8_W7.62mm_Socket, symbol L:ACS712xLCTR-05B
- added U5: LM2576HVS-5.0 29V-5V, Package_TO_SOT_SMD:TO-263-5_TabPin3, symbol L:LM2596T-12
- C1: value 220u 50V -> 2u2; footprint Capacitor_THT:CP_Radial_D10.0mm_P5.00mm -> Capacitor_THT:C_Disc_D5.0mm_W2.5mm_P5.00mm
- C2: value 220u 10V -> 100n; footprint Capacitor_THT:CP_Radial_D8.0mm_P3.50mm -> Capacitor_THT:C_Disc_D5.0mm_W2.5mm_P5.00mm
- C3: value 2u2 -> 1n
- C4: value 100n -> 220u 50V; footprint Capacitor_THT:C_Disc_D5.0mm_W2.5mm_P5.00mm -> Capacitor_THT:CP_Radial_D10.0mm_P5.00mm
- C5: value 1n -> 220u 10V; footprint Capacitor_THT:C_Disc_D5.0mm_W2.5mm_P5.00mm -> Capacitor_THT:CP_Radial_D8.0mm_P3.50mm
- D3: value allows down -> flyback
- D4: renamed from U1; value LM2596HV 29V-5V -> 33V bidir; footprint Package_TO_SOT_THT:TO-220-5_Vertical -> Diode_THT:D_DO-15_P10.16mm_Horizontal; symbol L:LM2596T-12 -> L:D_TVS
- D5: value SB560 -> allows down; footprint Diode_THT:D_DO-201AD_P12.70mm_Horizontal -> Diode_THT:D_DO-35_SOD27_P7.62mm_Horizontal
- K1: renamed from D2; value flyback -> energized = UP (raises desk); footprint Diode_THT:D_DO-35_SOD27_P7.62mm_Horizontal -> Relay_THT:Relay_SPDT_Hongfa_JQC-3FF_0XX-1Z; symbol L:D -> L:Relay_SPDT
- K2: renamed from D6; value flyback -> energized = DOWN (lowers desk); footprint Diode_THT:D_DO-35_SOD27_P7.62mm_Horizontal -> Relay_THT:Relay_SPDT_Hongfa_JQC-3FF_0XX-1Z; symbol L:D -> L:Relay_SPDT
- R7: value 1k -> 100k
- TB1: renamed from TB3; footprint TerminalBlock:TerminalBlock_MaiXu_MX126-5.0-02P_1x02_P5.00mm -> TerminalBlock:TerminalBlock_Xinya_XY308-2.54-2P_1x02_P2.54mm_Horizontal
- TB2: renamed from TB4; footprint TerminalBlock:TerminalBlock_MaiXu_MX126-5.0-02P_1x02_P5.00mm -> TerminalBlock:TerminalBlock_Xinya_XY308-2.54-2P_1x02_P2.54mm_Horizontal
- renumbered J3 to J1, R4 to R1, R5 to R2, R11 to R3, R14 to R4, R13 to R5, R15 to R6, U2 to U1
Connections:
- net +29V_RAW: now also C4.1, J3.3 (Pin_3), TB5.1 (Pin_1), U5.1 (VIN); no longer C1.1
- net +3V3: now also SW3.1 (A), SW4.1 (A)
- net +5V: now also C5.1, D3.1 (K), K1.A2, K2.A2, R7.1, D2.1 (K), Q1.1 (C), U2.16 (VCC), U2.2 (B), U2.3 (Clr), U3.14 (VCC), U4.8 (VCC), U5.2 (OUT), U5.4 (FB); no longer C4.1, D4.2 (OUT), D4.4 (FB), K1.1 (K), K2.1 (K)
- net DIR_A: now also R8.1, U3.2
- net DIR_B: now also R9.1, U3.5
- net DRV_UP: now also K1.11, U4.3 (IP-), U4.4 (IP-)
- net GND: now also C1.1, C3.2, D4.2 (A2), J3.4 (Pin_4), Q2.1 (C), Q4.3 (S), Q5.3 (S), R10.2, R8.2, R9.2, SW3.3 (C), SW4.3 (C), TB5.2 (Pin_2), U2.8 (GND), U3.7 (GND), U4.5 (GND), U5.3 (GND), U5.5 (~{ON}/OFF); no longer C1.2, C3.1, D4.3 (GND), D4.5 (~{ON}/OFF)
- net HND_A: now also SW4.2 (B)
- net HND_B: now also SW3.2 (B)
- net KICK: now also U2.1 (A)
- net MOT_A: now also D5.1 (K), K2.11, J3.1 (Pin_1), SW1.2 (B), TB4.1 (Pin_1); no longer D3.1 (K)
- net MOT_B: now also D6.1 (K), J3.2 (Pin_2), SW2.2 (B), TB4.2 (Pin_2), U4.1 (IP+), U4.2 (IP+)
- net MRET: now also K1.14, K2.14, D1.2 (A), Q5.2 (D); no longer D5.2 (A)
- net PWM: now also R10.1, U3.10
- net SCL: now also U1.38 (GPIO41/MTDI), TB3.2 (Pin_2); no longer U1.19 (GPIO13/ADC2_CH2)
- net SDA: now also U1.35 (GPIO38), TB3.1 (Pin_1); no longer U1.18 (GPIO12/ADC2_CH1)
- net VIOUT: now also U4.7 (VIOUT)
- net VSW: now also K1.12, K2.12, D1.1 (K); no longer D5.1 (K)
- net WDOG: now also U2.13 (Q), U3.1, U3.4, U3.9
- net at D3.2 (A): now also K2.A1, Q4.2 (D); no longer M1.1 (+)
- net at R7.2: now also C1.2, U2.14 (Cext), U2.15 (RCext)
- net at M1.2 (-): now also D6.2 (A), SW2.1 (A)
- net at Q3.1 (G): now also U3.3
- net at Q3.2 (D): now also K1.A1, D2.2 (A); no longer K2.2 (A)
- new net: R11.1, U3.8
- new net: C3.1, U4.6 (FILTER)
- new net: Q1.2 (B), Q2.2 (B), R11.2
- new net: Q1.3 (E), Q2.3 (E), Q5.1 (G)
- new net: Q4.1 (G), U3.6
- new net: D5.2 (A), M1.1 (+), SW1.1 (A)
